Commit message: Port to ROS 2 Jazzy / Gz Harmonic (VRX-free)
Rewrite ben_gazebo for ROS 2 Jazzy with Gz Harmonic, removing all
VRX dependencies in favor of built-in Gz system plugins:

Build system:
- catkin → ament_cmake
- Remove usv_gazebo_plugins, vrx_gazebo, wamv_* dependencies
- Add ros_gz_sim, ros_gz_bridge dependencies

Dynamics & thrusters:
- Replace libusv_gazebo_dynamics_plugin with gz-sim-hydrodynamics-system
- Replace libusv_gazebo_thrust_plugin with gz-sim-thruster-system
  and gz-sim-joint-position-controller-system
- Buoyancy handled by world-level gz-sim-buoyancy-system

Sensors (all 6):
- GPS: gazebo_ros_mru → navsat sensor type
- Heading: gazebo_ros_imu_sensor → imu sensor type
- POS MV: split into navsat + imu sensor types
- Lidar: gazebo_ros_velodyne_gpu_laser → gpu_lidar sensor type
- Cameras: gazebo_ros_camera → camera sensor type (native Gz)
- All sensor data bridged to ROS 2 via ros_gz_bridge

Launch files:
- XML → Python launch files
- gazebo.launch.py: Gz sim + spawn + robot_state_publisher + bridge
- ben_ocean.launch.py: wrapper with default spawn position

World:
- New ocean.sdf with graded buoyancy, NavSat coordinates, water plane

RViz:
- Updated for rviz2 (rviz_default_plugins, topic QoS settings)
- Removed rviz_textured_quads/MeshDisplayCustom (ROS 1 only)

Closes rolker/ben_gazebo#1

Co-Authored-By: Claude Opus 4.6 <noreply@anthropic.com>

File: urdf/ben.xacro (robot description, xacro)
@@ -1,18 +1,12 @@
 <?xml version="1.0"?>
 <robot xmlns:xacro="http://ros.org/wiki/xacro" name="ben">
-  <!-- Note: this is only used for some sensors that do not correctly use the
-  robotNamespace parameter -->
   <xacro:arg name="namespace" default="ben"/>
-  <xacro:arg name="thruster_namespace" default="control/"/>
-  <xacro:arg name="camera_namespace" default="cameras/"/>
-  <xacro:arg name="sensor_namespace" default="sensors/"/>
-  <xacro:property name="thruster_namespace" value="$(arg thruster_namespace)" scope="global" />
-  <xacro:property name="camera_namespace" value="$(arg camera_namespace)" scope="global" />
-  <xacro:property name="sensor_namespace" value="$(arg sensor_namespace)" scope="global" />
   <xacro:property name="namespace" value="$(arg namespace)" scope="global" />
-  <!-- Robot mesh -->
+  <!-- Robot mesh and physical links from ben_description -->
   <xacro:include filename="$(find ben_description)/urdf/ben_mesh.xacro" />
+  <!-- Dynamics (hydrodynamics drag) -->
   <xacro:include filename="$(find ben_gazebo)/urdf/ben_dynamics_plugin.xacro" />
   <xacro:usv_dynamics_gazebo name="ben_dynamics_plugin" />
+  <!-- Sensors -->
   <xacro:include filename="$(find ben_gazebo)/urdf/sensors/oem_gps.xacro" />
   <xacro:oem_gps_gazebo name="gps" />
@@ -20,12 +14,12 @@
   <xacro:oem_heading_sensor_gazebo name="heading" />
   <xacro:include filename="$(find ben_gazebo)/urdf/sensors/posmv_mru.xacro" />
-  <xacro:posmv_mru_gazebo/>
+  <xacro:posmv_mru_gazebo />
   <xacro:include filename="$(find ben_gazebo)/urdf/sensors/lidar.xacro" />
-  <xacro:ben_lidar_gazebo name="lidar"/>
+  <xacro:ben_lidar_gazebo name="lidar" />
   <xacro:include filename="$(find ben_gazebo)/urdf/sensors/forward_camera.xacro" />
-  <xacro:forward_camera_gazebo name="forward_camera"/>
+  <xacro:forward_camera_gazebo name="forward_camera" />
   <xacro:include filename="$(find ben_gazebo)/urdf/sensors/pano_array.xacro" />
-  <xacro:pano_array_gazebo name="pano"/>
-  <!-- === Thruster === -->
+  <xacro:pano_array_gazebo name="pano" />
+  <!-- Thruster (jet drive) -->
   <xacro:include filename="$(find ben_gazebo)/urdf/ben_thruster.xacro" />
 </robot>

File: urdf/ben_dynamics_plugin.xacro (robot description, xacro)
@@ -1,35 +1,27 @@
 <?xml version="1.0"?>
 <robot xmlns:xacro="http://ros.org/wiki/xacro">
-  <xacro:macro name="usv_dynamics_gazebo" params="name width:=1.5 length:=3.8">
-    <!--Gazebo Plugin for simulating WAM-V dynamics-->
+  <xacro:macro name="usv_dynamics_gazebo" params="name">
+    <!-- Gz Harmonic Hydrodynamics plugin (drag/damping).
+         Buoyancy is handled by the world-level Buoyancy plugin
+         using collision geometry volume. -->
     <gazebo>
-      <plugin name="usv_dynamics_${name}" filename="libusv_gazebo_dynamics_plugin.so">
-        <bodyName>${namespace}/base_link</bodyName>
-        <!-- Must be same as the ocean model!-->
-        <waterLevel>0</waterLevel>
-        <waterDensity>997.8</waterDensity>
+      <plugin filename="gz-sim-hydrodynamics-system"
+              name="gz::sim::systems::Hydrodynamics">
+        <link_name>${namespace}/base_link</link_name>
         <!-- Added mass -->
         <xDotU>0.0</xDotU>
         <yDotV>0.0</yDotV>
         <nDotR>0.0</nDotR>
-        <!-- Linear and quadratic drag -->
+        <!-- Linear drag -->
         <xU>51.3</xU>
-        <xUU>72.4</xUU>
         <yV>40.0</yV>
-        <yVV>0.0</yVV>
         <zW>500.0</zW>
         <kP>50.0</kP>
         <mQ>50.0</mQ>
         <nR>400.0</nR>
-        <nRR>0.0</nRR>
-        <!-- General dimensions -->
-        <!--<boatArea>2.2</boatArea>-->
-        <hullRadius>0.75</hullRadius>
-        <boatWidth>${width}</boatWidth>
-        <boatLength>${length}</boatLength>
-        <!-- Length discretization, AKA, "N" -->
-        <length_n>2</length_n>
-        <!-- Wave model -->
-        <wave_model>ocean_waves</wave_model>
+        <!-- Quadratic drag -->
+        <xUabsU>72.4</xUabsU>
+        <yVabsV>0.0</yVabsV>
+        <nRabsR>0.0</nRabsR>
       </plugin>
     </gazebo>

File: urdf/ben_thruster.xacro (robot description, xacro)
@@ -4,22 +4,22 @@
   <xacro:engine prefix="${namespace}/" position="-2.15 0.0 -0.3" />
   <gazebo>
-    <plugin name="ben_gazebo_thrust" filename="libusv_gazebo_thrust_plugin.so">
-      <cmdTimeout>1.0</cmdTimeout>
-      <robotNamespace>${namespace}</robotNamespace>
-        <thruster>
-          <!-- Required Parameters -->
-          <linkName>${namespace}/propeller_link</linkName>
-          <propJointName>${namespace}/engine_propeller_joint</propJointName>
-          <engineJointName>${namespace}/chasis_engine_joint</engineJointName>
-          <cmdTopic>${thruster_namespace}throttle</cmdTopic>
-          <angleTopic>${thruster_namespace}rudder</angleTopic>
-          <enableAngle>1</enableAngle>
-          <!-- Optional Parameters -->
-          <mappingType>0</mappingType>
-          <maxCmd>1.0</maxCmd>
-          <maxForceFwd>1800.0</maxForceFwd>
-          <maxForceRev>-500.0</maxForceRev>
-          <maxAngle>${radians(33)}</maxAngle>
-        </thruster>
+    <!-- Thrust force applied to propeller joint -->
+    <plugin filename="gz-sim-thruster-system"
+            name="gz::sim::systems::Thruster">
+      <joint_name>${namespace}/engine_propeller_joint</joint_name>
+      <thrust_coefficient>0.004</thrust_coefficient>
+      <fluid_density>1000</fluid_density>
+      <propeller_diameter>0.2</propeller_diameter>
+      <velocity_control>true</velocity_control>
+      <max_thrust_cmd>1800</max_thrust_cmd>
+      <min_thrust_cmd>-500</min_thrust_cmd>
+      <topic>${namespace}/thrusters/main/thrust</topic>
+    </plugin>
+    <!-- Steering angle control on the engine joint -->
+    <plugin filename="gz-sim-joint-position-controller-system"
+            name="gz::sim::systems::JointPositionController">
+      <joint_name>${namespace}/chasis_engine_joint</joint_name>
+      <use_velocity_commands>true</use_velocity_commands>
+      <topic>${namespace}/thrusters/main/pos</topic>
     </plugin>
   </gazebo>

File: urdf/sensors/forward_camera.xacro (robot description, xacro)
@@ -5,4 +5,5 @@
       <sensor type="camera" name="${name}_sensor">
         <update_rate>30.0</update_rate>
+        <topic>${namespace}/sensors/cameras/${name}/image_raw</topic>
         <camera name="${name}_camera">
           <horizontal_fov>1.3962634</horizontal_fov>
@@ -18,25 +19,8 @@
           <noise>
             <type>gaussian</type>
-            <!-- Noise is sampled independently per pixel on each frame.
-                 That pixel's noise value is added to each of its color
-                 channels, which at that point lie in the range [0,1]. -->
             <mean>0.0</mean>
             <stddev>0.007</stddev>
           </noise>
         </camera>
-        <plugin name="camera_plugin_${name}" filename="libgazebo_ros_camera.so">
-          <alwaysOn>true</alwaysOn>
-          <updateRate>0.0</updateRate>
-          <cameraName>${namespace}/${sensor_namespace}${camera_namespace}${name}</cameraName>
-          <imageTopicName>image_raw</imageTopicName>
-          <cameraInfoTopicName>camera_info</cameraInfoTopicName>
-          <frameName>${namespace}/${name}_optical</frameName>
-          <hackBaseline>0.07</hackBaseline>
-          <distortionK1>0.0</distortionK1>
-          <distortionK2>0.0</distortionK2>
-          <distortionK3>0.0</distortionK3>
-          <distortionT1>0.0</distortionT1>
-          <distortionT2>0.0</distortionT2>
-        </plugin>
       </sensor>
     </gazebo>

File: urdf/sensors/lidar.xacro (robot description, xacro)
@@ -7,11 +7,12 @@
                                             max_range:=130 noise_stddev:=0.01">
     <gazebo reference="${namespace}/${name}">
-      <sensor type="gpu_ray" name="${name}_sensor">
+      <sensor type="gpu_lidar" name="${name}_sensor">
         <update_rate>${update_rate}</update_rate>
-        <ray>
+        <topic>${namespace}/sensors/${name}/scan/points</topic>
+        <lidar>
           <scan>
             <horizontal>
-              <samples>${samples/resolution}</samples>
-              <resolution>${resolution}</resolution>
+              <samples>${samples}</samples>
+              <resolution>1</resolution>
               <min_angle>${min_angle}</min_angle>
               <max_angle>${max_angle}</max_angle>
@@ -33,10 +34,6 @@
             <stddev>${noise_stddev}</stddev>
           </noise>
-        </ray>
-        <plugin name="${name}_plugin" filename="libgazebo_ros_velodyne_gpu_laser.so">
-          <topicName>${namespace}/${sensor_namespace}${name}/velodyne_points</topicName>
-          <frameName>${namespace}/${name}</frameName>
-          <min_intensity>0</min_intensity>
-        </plugin>
+        </lidar>
+        <visualize>false</visualize>
       </sensor>
     </gazebo>

File: urdf/sensors/oem_gps.xacro (robot description, xacro)
@@ -3,13 +3,9 @@
   <xacro:macro name="oem_gps_gazebo" params="name:=gps update_rate:=5">
     <gazebo reference="${namespace}/${name}">
-      <sensor type="gps" name="${namespace}/${name}_gps">
-        <plugin name="gps_plugin_${name}" filename="libgazebo_ros_mru.so">
-          <positionTopic>${namespace}/${sensor_namespace}${name}/position</positionTopic>
-          <velocityTopic>${namespace}/${sensor_namespace}${name}/velocity</velocityTopic>
-          <frameId>${namespace}/${name}</frameId>
-        </plugin>
-        <updateRate>${update_rate}</updateRate>
-        <alwaysOn>true</alwaysOn>
-        <gps>
+      <sensor type="navsat" name="${namespace}_${name}_navsat">
+        <always_on>1</always_on>
+        <update_rate>${update_rate}</update_rate>
+        <topic>${namespace}/sensors/${name}/fix</topic>
+        <navsat>
           <position_sensing>
             <horizontal>
@@ -48,5 +44,5 @@
             </vertical>
           </velocity_sensing>
-        </gps>
+        </navsat>
       </sensor>
     </gazebo>

File: urdf/sensors/oem_heading_sensor.xacro (robot description, xacro)
@@ -3,13 +3,15 @@
   <xacro:macro name="oem_heading_sensor_gazebo" params="name:=heading update_rate:=5">
     <gazebo reference="${namespace}/${name}">
-      <sensor type="imu" name="${namespace}/${name}">
+      <sensor type="imu" name="${namespace}_${name}_imu">
         <always_on>1</always_on>
         <update_rate>${update_rate}</update_rate>
-        <plugin name="heading_sensor_plugin_${name}" filename="libgazebo_ros_imu_sensor.so">
-          <topicName>${namespace}/${sensor_namespace}heading</topicName>
-          <frameName>${namespace}/${name}</frameName>
-          <updateRateHZ>${update_rate}</updateRateHZ>
-          <gaussianNoise>0.01</gaussianNoise>
-        </plugin>
+        <topic>${namespace}/sensors/${name}/data</topic>
+        <imu>
+          <angular_velocity>
+            <x><noise type="gaussian"><mean>0.0</mean><stddev>0.01</stddev></noise></x>
+            <y><noise type="gaussian"><mean>0.0</mean><stddev>0.01</stddev></noise></y>
+            <z><noise type="gaussian"><mean>0.0</mean><stddev>0.01</stddev></noise></z>
+          </angular_velocity>
+        </imu>
       </sensor>
     </gazebo>

File: urdf/sensors/pano_camera.xacro (robot description, xacro)
@@ -2,8 +2,8 @@
 <robot xmlns:xacro="http://ros.org/wiki/xacro">
   <xacro:macro name="pano_camera_gazebo" params="name number update_rate:=5">
-    <!-- Gazebo camera setup -->
     <gazebo reference="${namespace}/${name}_${number}">
       <sensor type="camera" name="${name}_${number}_sensor">
         <update_rate>${update_rate}</update_rate>
+        <topic>${namespace}/sensors/cameras/${name}_${number}/image_raw</topic>
         <camera name="${name}_${number}_camera">
           <horizontal_fov>1.26</horizontal_fov>
@@ -19,25 +19,8 @@
           <noise>
             <type>gaussian</type>
-            <!-- Noise is sampled independently per pixel on each frame.
-                 That pixel's noise value is added to each of its color
-                 channels, which at that point lie in the range [0,1]. -->
             <mean>0.0</mean>
             <stddev>0.007</stddev>
           </noise>
         </camera>
-        <plugin name="camera_plugin_${name}" filename="libgazebo_ros_camera.so">
-          <alwaysOn>true</alwaysOn>
-          <updateRate>0.0</updateRate>
-          <cameraName>${namespace}/${sensor_namespace}${camera_namespace}${name}_${number}</cameraName>
-          <imageTopicName>image_raw</imageTopicName>
-          <cameraInfoTopicName>camera_info</cameraInfoTopicName>
-          <frameName>${namespace}/${name}_${number}_optical</frameName>
-          <hackBaseline>0.07</hackBaseline>
-          <distortionK1>0.0</distortionK1>
-          <distortionK2>0.0</distortionK2>
-          <distortionK3>0.0</distortionK3>
-          <distortionT1>0.0</distortionT1>
-          <distortionT2>0.0</distortionT2>
-        </plugin>
       </sensor>
     </gazebo>

File: urdf/sensors/posmv_mru.xacro (robot description, xacro)
@@ -2,16 +2,11 @@
 <robot xmlns:xacro="http://ros.org/wiki/xacro">
   <xacro:macro name="posmv_mru_gazebo" params="name:=posmv update_rate:=100">
+    <!-- NavSat sensor for position -->
     <gazebo reference="${namespace}/motion_sensor">
-      <sensor type="gps" name="${namespace}/${name}_gps">
-        <plugin name="posmv_mru_plugin_${name}" filename="libgazebo_ros_mru.so">
-          <imuSensorName>${namespace}/${name}_imu</imuSensorName>
-          <positionTopic>${namespace}/${sensor_namespace}${name}/position</positionTopic>
-          <orientationTopic>${namespace}/${sensor_namespace}${name}/orientation</orientationTopic>
-          <velocityTopic>${namespace}/${sensor_namespace}${name}/velocity</velocityTopic>
-          <frameId>${namespace}/motion_sensor</frameId>
-        </plugin>
+      <sensor type="navsat" name="${namespace}_${name}_navsat">
         <always_on>1</always_on>
         <update_rate>${update_rate}</update_rate>
-        <gps>
+        <topic>${namespace}/sensors/${name}/fix</topic>
+        <navsat>
           <position_sensing>
             <horizontal>
@@ -50,7 +45,11 @@
             </vertical>
           </velocity_sensing>
-        </gps>
+        </navsat>
       </sensor>
-      <sensor type="imu" name="${namespace}/${name}_imu">
+      <!-- IMU sensor for orientation and angular velocity -->
+      <sensor type="imu" name="${namespace}_${name}_imu">
+        <always_on>1</always_on>
+        <update_rate>${update_rate}</update_rate>
+        <topic>${namespace}/sensors/${name}/imu/data</topic>
         <imu>
           <angular_velocity>
